Commit message: update symmetry-aware grasping demo

File: ros/examples/symaware_grasp/urdf/simple_six_dof_arm.urdf (robot description, URDF)
Before this commit: robot simple_six_dof_arm, 8 links, 7 joints
Links:
- link tool0: mass 0.3 -> 0.7; geometry collision box size=0.04 0.17 0.12; collision box size=0.13 0.025 0.14

Commit message: Add bottle grasp distribution comparison recordings
Record the same bottle grasp with axial Bingham symmetry and a single-pose
Bingham distribution at a bottle yaw of 3*pi/8. Save synchronized oblique,
top and side-by-side RViz movies with TCP axes, rosbag, CSV, graphs, models
and the instructions needed to reproduce and analyze both conditions.

Shorten the flange to keep it outside the bottle and use an elevated
transfer followed by a straight approach. Check conservative bottle
clearance during planning, execution and independent bag analysis. Add
movable jaws and keep the configured bottle reference frame consistent
across both distributions.

Validation: 45 symaware_grasp tests passed; both recorded trials reached
their grasp with positive clearance; individual and combined videos have
matching frame counts; bag reanalysis reproduces the complete CSV and
summary for both conditions.

File: ros/examples/symaware_grasp/urdf/simple_six_dof_arm.urdf (robot description, URDF)
Before this commit: robot simple_six_dof_arm, 8 links, 7 joints
Links:
- link link_6: geometry collision cylinder length=0.025 radius=0.032; visual cylinder length=0.025 radius=0.032
